Commit message: updated model and cleaning

File: urdf/nao.urdf (robot description, URDF)
Before this commit: robot naoH25V40, 50 links, 49 joints
Links:
- removed link LFeet
- removed link LSonar
- removed link RFeet
- removed link RSonar
- added link CameraBottom_frame
- added link ChestButton_frame
- added link HeadTouchFront_frame
- added link HeadTouchMiddle_frame
- added link HeadTouchRear_frame
- added link ImuAccelerometer_frame
- added link ImuGyrometer_frame
- added link LFootBumperLeft_frame
- added link LFootBumperRight_frame
- added link LFsrFL_frame
- added link LFsrFR_frame
- added link LFsrRL_frame
- added link LFsrRR_frame
- added link LHandTouchBack_frame
- added link LHandTouchLeft_frame
- added link LHandTouchRight_frame
- added link LInfraRed_frame
- added link LSonar_frame
- added link RFootBumperLeft_frame
- added link RFootBumperRight_frame
- added link RFsrFL_frame
- added link RFsrFR_frame
- added link RFsrRL_frame
- added link RFsrRR_frame
- added link RHandTouchBack_frame
- added link RHandTouchLeft_frame
- added link RHandTouchRight_frame
- added link RInfraRed_frame
- added link RSonar_frame
- link l_sole: mass None -> 0.16184; geometry collision mesh filename=package://nao_meshes/meshes/V40/collision/LAnkleRoll.stl scale=0.1 0.1 0.1; visual mesh filename=package://nao_meshes/meshes/V40/visual/LAnkleRoll.dae scale=0.1 0.1 0.1
- link r_sole: mass None -> 0.16184; geometry collision mesh filename=package://nao_meshes/meshes/V40/collision/RAnkleRoll.stl scale=0.1 0.1 0.1; visual mesh filename=package://nao_meshes/meshes/V40/visual/RAnkleRoll.dae scale=0.1 0.1 0.1
Joints:
- removed joint l_sole_joint
- removed joint r_sole_joint
- added joint CameraBottom_joint: type fixed, parent Head, child CameraBottom_frame, origin xyz=0.05071 0 0.01774 rpy=0 0.6929 0
- added joint ChestButton_joint: type fixed, parent torso, child ChestButton_frame, origin xyz=0.049871 0.001588 0.055163 rpy=0 0 0
- added joint HeadTouchFront_joint: type fixed, parent Head, child HeadTouchFront_frame, origin xyz=0.0312 0 0.1014 rpy=0 -1.186099535 0
- added joint HeadTouchMiddle_joint: type fixed, parent Head, child HeadTouchMiddle_frame, origin xyz=0.001 0 0.1099 rpy=0 -1.57079632679 0
- added joint HeadTouchRear_joint: type fixed, parent Head, child HeadTouchRear_frame, origin xyz=-0.0257 0 0.1045 rpy=3.14159265359 -1.333192995 3.14159265359
- added joint ImuAccelerometer_joint: type fixed, parent torso, child ImuAccelerometer_frame, origin xyz=-0.008 0.00606 0.027 rpy=0 0 0
- added joint ImuGyrometer_joint: type fixed, parent torso, child ImuGyrometer_frame, origin xyz=-0.008 -0.006 0.029 rpy=0 0 0
- added joint LFootBumperLeft_joint: type fixed, parent l_ankle, child LFootBumperLeft_frame, origin xyz=0.0876 0.019 -0.035 rpy=0 0 0
- added joint LFootBumperRight_joint: type fixed, parent l_ankle, child LFootBumperRight_frame, origin xyz=0.0876 -0.014 -0.035 rpy=0 0 0
- added joint LFsrFL_joint: type fixed, parent l_ankle, child LFsrFL_frame, origin xyz=0.07025 0.0299 0 rpy=0 0 0
- added joint LFsrFR_joint: type fixed, parent l_ankle, child LFsrFR_frame, origin xyz=0.07025 -0.0231 0 rpy=0 0 0
- added joint LFsrRL_joint: type fixed, parent l_ankle, child LFsrRL_frame, origin xyz=-0.03025 0.0299 0 rpy=0 0 0
- added joint LFsrRR_joint: type fixed, parent l_ankle, child LFsrRR_frame, origin xyz=-0.02965 -0.0191 0 rpy=0 0 0
- added joint LHandTouchBack_joint: type fixed, parent l_wrist, child LHandTouchBack_frame, origin xyz=0.038 0 0.025 rpy=0 -1.57079632679 0
- added joint LHandTouchLeft_joint: type fixed, parent l_wrist, child LHandTouchLeft_frame, origin xyz=0.032 0.025 0.003 rpy=0 0 0
- added joint LHandTouchRight_joint: type fixed, parent l_wrist, child LHandTouchRight_frame, origin xyz=0.035 -0.025 0.0035 rpy=0 0 0
- added joint LInfraRed_joint: type fixed, parent Head, child LInfraRed_frame, origin xyz=0.0441 0.0257 0.0466 rpy=0 0 0
- added joint RFootBumperLeft_joint: type fixed, parent r_ankle, child RFootBumperLeft_frame, origin xyz=0.0876 0.014 -0.035 rpy=0 0 0
- added joint RFootBumperRight_joint: type fixed, parent r_ankle, child RFootBumperRight_frame, origin xyz=0.0876 -0.019 -0.035 rpy=0 0 0
- added joint RFsrFL_joint: type fixed, parent r_ankle, child RFsrFL_frame, origin xyz=0.07025 0.0231 0 rpy=0 0 0
- added joint RFsrFR_joint: type fixed, parent r_ankle, child RFsrFR_frame, origin xyz=0.07025 -0.0299 0 rpy=0 0 0
- added joint RFsrRL_joint: type fixed, parent r_ankle, child RFsrRL_frame, origin xyz=-0.03025 0.0191 0 rpy=0 0 0
- added joint RFsrRR_joint: type fixed, parent r_ankle, child RFsrRR_frame, origin xyz=-0.02965 -0.0299 0 rpy=0 0 0
- added joint RHandTouchBack_joint: type fixed, parent r_wrist, child RHandTouchBack_frame, origin xyz=0.038 0 0.025 rpy=0 -1.57079632679 0
- added joint RHandTouchLeft_joint: type fixed, parent r_wrist, child RHandTouchLeft_frame, origin xyz=0.032 0.025 0.003 rpy=0 0 0
- added joint RHandTouchRight_joint: type fixed, parent r_wrist, child RHandTouchRight_frame, origin xyz=0.035 -0.025 0.0035 rpy=0 0 0
- added joint RInfraRed_joint: type fixed, parent Head, child RInfraRed_frame, origin xyz=0.0441 -0.0257 0.0466 rpy=0 0 0
- joint CameraTop_joint: origin xyz=0.0539 0 0.0679 rpy=0 0 0 -> xyz=0.05871 0 0.06364 rpy=0 0.0209 0
- joint LAnkleRoll: child LFeet -> l_sole
- joint LSonar_joint: child LSonar -> LSonar_frame; origin xyz=0.0507 0.03785 0.06035 rpy=0 0.04365 -0.39265 -> xyz=0.0507 0.03785 0.06035 rpy=0 0.04365 0.39265
- joint RAnkleRoll: child RFeet -> r_sole
- joint RSonar_joint: child RSonar -> RSonar_frame; origin xyz=0.0507 -0.03785 0.06035 rpy=0 0.04365 0.39265 -> xyz=0.0507 -0.03785 0.06035 rpy=0 0.04365 -0.39265
- joint gaze_joint: origin xyz=0 0 0 rpy=0 0 0 -> xyz=0.05871 0 0.06364 rpy=0 0.0209 0; parent CameraTop_frame -> Head
